File: Placa Junio/PlacaJunio/PlacaJunio.kicad_sch (KiCad schematic)
At the start: 20 parts, among them J1 Bateria, J3 Terminal Drogue, J4 Terminal Drogue, Q2 IRLML0030, Q3 IRLML0030, Q4 IRLML0030, U1 L80-R, U4 MODULO MICRO SD, U6 LM1117MP-3.3V

Commit message: d
Parts:
- removed J3, J4: Terminal Drogue, TerminalBlock:TerminalBlock_bornier-2_P5.08mm, symbol Connector:Screw_Terminal_01x02
- removed Q2, Q3: IRLML0030, Package_TO_SOT_SMD:SOT-23, symbol Transistor_FET:IRLML0030
- removed R5, R7: 10k, Resistor_SMD:R_0402_1005Metric, symbol Device:R
- removed R6, R8: 4.7 Ohm, 2.5W max, Resistor_THT:R_Axial_DIN0204_L3.6mm_D1.6mm_P2.54mm_Vertical, symbol Device:R
- removed U6: LM1117MP-3.3V, Package_TO_SOT_SMD:SOT-223-3_TabPin2, symbol Regulator_Linear:LM1117MP-3.3
- added U5: TSR2-2433N, Converter_DCDC:Converter_DCDC_TRACO_TSR2-24xxN_TSR2-24xxxN_THT, symbol Regulator_Switching:TSR2-2433N
Connections:
- net +3V3: now also U5.3 (Vout)
- net +BATT: now also U5.1 (Vin)
- net GND: now also U5.2 (GND)
Other:
- added sheet Screw_Terminals (Screw_Terminals.kicad_sch)
- note removed: "Activador de paracaídas"
- moved on the sheet: C5

Commit message: Cambios PCB
Parts:
- removed U1: L80-R, RF_GPS:Quectel_L80-R, symbol RF_GPS:L80-R
- added C7: 100nF, Capacitor_SMD:C_1206_3216Metric_Pad1.33x1.80mm_HandSolder, symbol Device:C_Polarized_US
- added IC1: LC86LICMD, LC86LICMD, symbol LC86LICMD:LC86LICMD
Connections:
- net +3V3: now also C7.1, IC1.4 (VCC)
- net GND: now also C7.2, IC1.12 (GND_2), IC1.3 (GND_1)
- net RX_GPS: now also IC1.1 (RXD)
- net TX_GPS: now also IC1.2 (TXD)
- no-connect marks 10 -> 12
Other:
- moved on the sheet: C6

Commit message: Cambios
Other:
- note added: "QUITAR BOTÓN RESET"
Changed lines of the file:
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@@
+		)
+	)
+	(text "QUITAR BOTÓN RESET\n"
+		(exclude_from_sim no)
+		(at 125.476 114.3 0)
+		(effects
+			(font
+				(size 1.27 1.27)
+			)
 		)
 	)

Commit message: Cambios
Connections:
- net Buzzer: now also U2.4 (A0)
- net MISO: now also U2.28 (D10)
- net MOSI: now also U2.29 (D11)
- net SCK: now also U2.30 (D12)
- net SD_CS: now also U2.1 (D_13)
- net RX_LoRa: now reaches U2.20 (D2)
- net RX_LoRa: now also U3.3 (RX)
- net TX_LoRa: now reaches U2.21 (D3)
- net TX_LoRa: now also U3.4 (TX)
- net M1_LoRa: now reaches U2.22 (D4)
- net M1_LoRa: now also U3.2 (M1)
- net M0_LoRa: now reaches U2.23 (D5)
- net M0_LoRa: now also U3.1 (M0)
- net PARACAIDAS 1: now reaches U2.24 (D6)
- net PARACAIDAS 2: now reaches U2.25 (D7)
- net PARACAIDAS 3: now reaches U2.26 (D8)
- net PARACAIDAS 4: now reaches U2.27 (D9)
- net SENSE 1: now reaches U2.5 (A1)
- net SENSE 2: now reaches U2.6 (A2)
- net SENSE 3: now reaches U2.7 (A3)
- net SENSE 4: now reaches U2.8 (A4)
- no-connect marks 12 -> 13
Other:
- sheet Screw_Terminals ports: added SENSE1, SENSE2, SENSE3, SENSE4; removed none

Commit message: Update Placa
Parts:
- removed U2: ~, Cohete_Julio:Nano BLE 33 Sense, symbol CoheteJulio:Nano_33_BLE_Sense
- added U1: ~, symbol CoheteJulio:Nano_33_BLE_Sense
- IC1: footprint LC86LICMD -> Cohete_Julio:LC86LICMD
Connections:
- net +3V3: now also U1.2 (+3v3)
- net Buzzer: now also U1.4 (A0)
- net GND: now also U1.14 (GND), U1.19 (GND)
- net M0_LoRa: now also U1.23 (D5)
- net M1_LoRa: now also U1.22 (D4)
- net MISO: now also U1.28 (D10)
- net MOSI: now also U1.29 (D11)
- net PARACAIDAS 1: now also U1.24 (D6)
- net PARACAIDAS 2: now also U1.25 (D7)
- net PARACAIDAS 3: now also U1.26 (D8)
- net PARACAIDAS 4: now also U1.27 (D9)
- net RX_GPS: now also U1.16 (TX)
- net RX_LoRa: now also U1.20 (D2)
- net SCK: now also U1.30 (D12)
- net SD_CS: now also U1.1 (D_13)
- net SENSE 1: now also U1.5 (A1)
- net SENSE 2: now also U1.6 (A2)
- net SENSE 3: now also U1.7 (A3)
- net SENSE 4: now also U1.8 (A4)
- net TX_GPS: now also U1.17 (RX)
- net TX_LoRa: now also U1.21 (D3)
- no-connect marks 13 -> 16

Commit message: cj
Connections:
- net +3V3: now also IC1.5 (V_BCKP)
- no-connect marks 16 -> 15
Other:
- note added: "Control Cargas pólvora"
- moved on the sheet: BZ1, C2, C5, C6, C7, IC1, J1, Q4, R9, U1, U3, U4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
