File: Placa Junio/PlacaJunio/PlacaJunio.kicad_pcb (KiCad board)
At the start: 2 copper layers, 35 x 113 mm, 30 parts, among them IC1 LC86LICMD, J1 Conn_01x07_Pin, J3 Terminal P2, J4 Terminal P1, J5 Terminal P3, J6 Terminal P4, Q2 IRLML0030, Q3 IRLML0030, Q4 IRLML0030, U5 TSR2-2433N

Commit message: V1 para producir ya, falta BOM
Parts:
- moved D1 1.88 mm to (148.2, 132.5)
- moved Q4 1.88 mm to (140.7, 134.6)
- moved R9 1.88 mm to (138.0, 134.5)
- moved BZ1 1.88 mm to (148.2, 139.0)
Connections:
- J5 pad 1: Net-(J5-Pin_1) -> GND
- J5 pad 2: GND -> /Armado
- J6 pad 2: Net-(J5-Pin_1) -> GND
- U1 pad 1: /Buzzer -> /Armado
- U1 pad 6: unconnected-(U1-A2-Pad6)_1 -> /Buzzer
Routing:
- net /Armado: track 0.00 -> 41.6 mm
- net +3V3: track 136.8 -> 159.4 mm, vias 0 -> 1
- net /Buzzer: track 75.9 -> 65.0 mm
- net /TX_GPS: track 36.1 -> 39.5 mm
- net /RX_GPS: track 37.6 -> 39.1 mm
- net GND: track 17.8 -> 17.0 mm
- net /SENSE 2: track 42.2 -> 42.0 mm, vias 2 -> 0
- net /PARACAIDAS 2: vias 4 -> 2
- net /PARACAIDAS 1: vias 6 -> 4
- net /SENSE 1: vias 2 -> 0
- removed copper zone on F.Cu, net Net-(J5-Pin_1)
