File: Placa Junio/PlacaJunio/PlacaJunio.kicad_pcb (KiCad board)
At the start: 2 copper layers, 35 x 113 mm, 30 parts, among them IC1 LC86LICMD, J1 Conn_01x07_Pin, J3 Terminal P2, J4 Terminal P1, J5 Terminal P3, J6 Terminal P4, Q2 IRLML0030, Q3 IRLML0030, Q4 IRLML0030, U5 TSR2-2433N

Commit message: No había guardado KiCAD lmao
Parts:
- renumbered C2 to C1, C5 to C2, C6 to C3, C7 to C4, J6 to J1, J5 to J2, J1 to J3, J3 to J5, Q4 to Q1, Q3 to Q2, Q2 to Q3, R9 to R1, R14 to R2, R17 to R3, R15 to R4, R18 to R5, R7 to R6, R5 to R7, U5 to U1, U3 to U2, U1 to U3, U2 to U4

Commit message: Casi me olvido de la serigrafía
Parts:
- added G***: LOGO, LOGO, F.Cu at (149.9, 55.0)
Other:
- board text added: "ADA V2.0"
- board text added: "Esta sí que sí ;)"
