File: Placa Junio/PlacaJunio/MicroSD.kicad_sch (KiCad schematic)
At the start: 1 part

Commit message: No había guardado KiCAD lmao
Parts:
- renumbered U2 to U4
Changed lines of the file:
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@@
 		(dnp no)
 		(fields_autoplaced yes)
-		(property "Reference" "U2"
+		(property "Reference" "U4"
 			(at 132.08 63.5 0)
 			(effects
@@
 			(project "PlacaJunio"
 				(path "/b66ba01b-450c-41a1-983e-895a21bf9603/5e6901b7-2508-4e4e-8a04-dcdebc2757da"
-					(reference "U2")
+					(reference "U4")
 					(unit 1)
 				)
@@
 		(dnp no)
 		(fields_autoplaced yes)
-		(property "Reference" "#PWR012"
+		(property "Reference" "#PWR022"
 			(at 127 68.58 0)
 			(effects
@@
 			(project "PlacaJunio"
 				(path "/b66ba01b-450c-41a1-983e-895a21bf9603/5e6901b7-2508-4e4e-8a04-dcdebc2757da"
-					(reference "#PWR012")
+					(reference "#PWR022")
 					(unit 1)
 				)
@@
 		(dnp no)
 		(fields_autoplaced yes)
-		(property "Reference" "#PWR017"
+		(property "Reference" "#PWR023"
 			(at 116.84 76.2 0)
 			(effects
@@
 			(project "PlacaJunio"
 				(path "/b66ba01b-450c-41a1-983e-895a21bf9603/5e6901b7-2508-4e4e-8a04-dcdebc2757da"
-					(reference "#PWR017")
+					(reference "#PWR023")
 					(unit 1)
 				)
