File: Placa Junio/PlacaJunio/Screw_Terminals.kicad_sch (KiCad schematic)
At the start: 10 parts, among them J3 Terminal P2, J4 Terminal P1, Q2 IRLML0030, Q3 IRLML0030

Commit message: No había guardado KiCAD lmao
Parts:
- renumbered J3 to J5, Q3 to Q2, Q2 to Q3, R14 to R2, R17 to R3, R15 to R4, R18 to R5, R7 to R6, R5 to R7
Changed lines of the file:
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@@
 		(on_board yes)
 		(dnp no)
-		(property "Reference" "Q3"
+		(property "Reference" "Q2"
 			(at 104.14 100.33 0)
 			(effects
@@
 			(project "PlacaJunio"
 				(path "/b66ba01b-450c-41a1-983e-895a21bf9603/7bf72e12-8d12-4e35-9fad-8768305749e5"
-					(reference "Q3")
+					(reference "Q2")
 					(unit 1)
 				)
@@
 		(dnp no)
 		(fields_autoplaced yes)
-		(property "Reference" "R5"
+		(property "Reference" "R7"
 			(at 133.35 101.6 0)
 			(effects
@@
 			(project "PlacaJunio"
 				(path "/b66ba01b-450c-41a1-983e-895a21bf9603/7bf72e12-8d12-4e35-9fad-8768305749e5"
-					(reference "R5")
+					(reference "R7")
 					(unit 1)
 				)
@@
 		(on_board yes)
 		(dnp no)
-		(property "Reference" "J3"
+		(property "Reference" "J5"
 			(at 148.59 77.47 0)
 			(effects
@@
 			(project "PlacaJunio"
 				(path "/b66ba01b-450c-41a1-983e-895a21bf9603/7bf72e12-8d12-4e35-9fad-8768305749e5"
-					(reference "J3")
+					(reference "J5")
 					(unit 1)
 				)
@@
 		(dnp no)
 		(fields_autoplaced yes)
-		(property "Reference" "R7"
+		(property "Reference" "R6"
 			(at 92.71 101.6 0)
 			(effects
@@
 			(project "PlacaJunio"
 				(path "/b66ba01b-450c-41a1-983e-895a21bf9603/7bf72e12-8d12-4e35-9fad-8768305749e5"
-					(reference "R7")
+					(reference "R6")
 					(unit 1)
 				)
@@
 		(dnp no)
 		(fields_autoplaced yes)
-		(property "Reference" "R18"
+		(property "Reference" "R5"
 			(at 158.75 99.0599 0)
 			(effects
@@
 			(project "PlacaJunio"
 				(path "/b66ba01b-450c-41a1-983e-895a21bf9603/7bf72e12-8d12-4e35-9fad-8768305749e5"
-					(reference "R18")
+					(reference "R5")
 					(unit 1)
 				)
@@
 		(on_board yes)
 		(dnp no)
-		(property "Reference" "#PWR05"
+		(property "Reference" "#PWR019"
 			(at 132.08 73.66 0)
 			(effects
@@
 			(project "PlacaJunio"
 				(path "/b66ba01b-450c-41a1-983e-895a21bf9603/7bf72e12-8d12-4e35-9fad-8768305749e5"
-					(reference "#PWR05")
+					(reference "#PWR019")
 					(unit 1)
 				)
@@
 		(on_board yes)
 		(dnp no)
-		(property "Reference" "#PWR06"
+		(property "Reference" "#PWR018"
 			(at 91.44 73.66 0)
 			(effects
@@
 			(project "PlacaJunio"
 				(path "/b66ba01b-450c-41a1-983e-895a21bf9603/7bf72e12-8d12-4e35-9fad-8768305749e5"
-					(reference "#PWR06")
+					(reference "#PWR018")
 					(unit 1)
 				)
@@
 		(dnp no)
 		(fields_autoplaced yes)
-		(property "Reference" "#PWR02"
+		(property "Reference" "#PWR020"
 			(at 100.33 113.03 0)
 			(effects
@@
 			(project "PlacaJunio"
 				(path "/b66ba01b-450c-41a1-983e-895a21bf9603/7bf72e12-8d12-4e35-9fad-8768305749e5"
-					(reference "#PWR02")
+					(reference "#PWR020")
 					(unit 1)
 				)
@@
 		(dnp no)
 		(fields_autoplaced yes)
-		(property "Reference" "R14"
+		(property "Reference" "R2"
 			(at 102.87 86.3599 0)
 			(effects
@@
 			(project "PlacaJunio"
 				(path "/b66ba01b-450c-41a1-983e-895a21bf9603/7bf72e12-8d12-4e35-9fad-8768305749e5"
-					(reference "R14")
+					(reference "R2")
 					(unit 1)
 				)
@@
 		(dnp no)
 		(fields_autoplaced yes)
-		(property "Reference" "R15"
+		(property "Reference" "R4"
 			(at 118.11 95.2499 0)
 			(effects
@@
 			(project "PlacaJunio"
 				(path "/b66ba01b-450c-41a1-983e-895a21bf9603/7bf72e12-8d12-4e35-9fad-8768305749e5"
-					(reference "R15")
+					(reference "R4")
 					(unit 1)
 				)
@@
 		(dnp no)
 		(fields_autoplaced yes)
-		(property "Reference" "R17"
+		(property "Reference" "R3"
 			(at 143.51 86.3599 0)
 			(effects
@@
 			(project "PlacaJunio"
 				(path "/b66ba01b-450c-41a1-983e-895a21bf9603/7bf72e12-8d12-4e35-9fad-8768305749e5"
-					(reference "R17")
+					(reference "R3")
 					(unit 1)
 				)
@@
 		(on_board yes)
 		(dnp no)
-		(property "Reference" "Q2"
+		(property "Reference" "Q3"
 			(at 144.78 100.33 0)
 			(effects
@@
 			(project "PlacaJunio"
 				(path "/b66ba01b-450c-41a1-983e-895a21bf9603/7bf72e12-8d12-4e35-9fad-8768305749e5"
-					(reference "Q2")
+					(reference "Q3")
 					(unit 1)
 				)
@@
 		(dnp no)
 		(fields_autoplaced yes)
-		(property "Reference" "#PWR03"
+		(property "Reference" "#PWR021"
 			(at 140.97 113.03 0)
 			(effects
@@
 			(project "PlacaJunio"
 				(path "/b66ba01b-450c-41a1-983e-895a21bf9603/7bf72e12-8d12-4e35-9fad-8768305749e5"
-					(reference "#PWR03")
-					(unit 1)
-				)
+					(reference "#PWR021")
+					(unit 1)
+				)
